Commit message: Added VLP16, Checked it works, Wrapped URDF into Xacro

File: src/osv_description/urdf/osv.urdf.xacro (robot description, xacro)
@@ -1,4 +1,10 @@
 <?xml version="1.0"?>
-<robot xmlns:xacro="http://ros.org/wiki/xacro" name="prius">
+<robot xmlns:xacro="http://ros.org/wiki/xacro" name="osv">
+  <!-- Add the correct Velodyne sensor-->
+  <xacro:include filename="$(find velodyne_description)/urdf/VLP-16.urdf.xacro"/>
+  <VLP-16 parent="base_link" name="velodyne" topic="/velodyne_points" hz="10" samples="440">
+    <origin xyz="0 0.4 1.8" rpy="0 0 0" />
+  </VLP-16>
+  <!-- TODO: Remove the old laser scanner-->
   <!--- Surface properties must come first? -->
   <gazebo reference="front_left_wheel">
@@ -249,5 +255,5 @@
   </joint>
   <!-- Sensor links and fixed joints -->
-  <link name="center_laser_link">
+  <!--link name="center_laser_link">
     <inertial>
       <mass value="1"/>
@@ -259,6 +265,6 @@
     <child link="center_laser_link"/>
     <origin xyz="0 0.4 1.8" rpy="0 0 -1.5707"/>
-  </joint>
-  <link name="front_left_laser_link">
+  </joint-->
+  <!--link name="front_left_laser_link">
     <inertial>
       <mass value="1"/>
@@ -281,5 +287,5 @@
     <child link="front_right_laser_link"/>
     <origin xyz="-1 -2.3 0.5" rpy="0 0.05 3.14"/>
-  </joint>
+  </joint-->
   <gazebo reference="base_link_connection">
     <disableFixedJointLumping>true</disableFixedJointLumping>
@@ -463,5 +469,5 @@
     </plugin>
   </gazebo>
-  <gazebo reference="center_laser_link">
+  <!--gazebo reference="center_laser_link">
     <sensor name='center_laser_sensor' type='ray'>
       <ray>
@@ -555,5 +561,5 @@
       <visualize>0</visualize>
     </sensor>
-  </gazebo>
+  </gazebo-->
   <gazebo reference="front_camera_link">
     <sensor type="camera" name="front_camera_sensor">
